Commit message: 提交更新的URDF文件

File: gluon_6l3_description/urdf/gluon_6l3_description_orAcolor.urdf (robot description, URDF)
Before this commit: robot gluon_6l3_description, 7 links, 6 joints
Links:
- added link tool0
Joints:
- added joint wrist_3_link-tool0_fixed_joint: type fixed, parent wrist_3_link, child tool0, origin xyz=0 0.04436 0 rpy=-1.57079632679 0 0

File: gluon_6l3_description/urdf/gluon_6l3_description_world(orColor).urdf (robot description, URDF)
Before this commit: robot gluon_6l3_description, 7 links, 6 joints
Links:
- added link base
- added link ee_link; collision box size=0.01 0.01 0.01
- added link tool0
- added link world
Joints:
- added joint base_link-base_fixed_joint: type fixed, parent base_link, child base, origin xyz=0 0 0 rpy=0 0 -3.1415926536
- added joint ee_fixed_joint: type fixed, parent wrist_3_link, child ee_link, origin xyz=0.0 0.04436 0.0 rpy=0.0 0.0 1.57079632679
- added joint world_joint: type fixed, parent world, child base_link, origin xyz=0.0 0.0 0.0 rpy=3.1415926536 3.1415926536 0.0
- added joint wrist_3_link-tool0_fixed_joint: type fixed, parent wrist_3_link, child tool0, origin xyz=0 0.04436 0 rpy=-1.57079632679 0 0

File: gluon_6l3_description/urdf/gluon_6l3_description_world.urdf (robot description, URDF)
Before this commit: robot gluon_6l3_description, 7 links, 6 joints
Links:
- added link base
- added link ee_link; collision box size=0.01 0.01 0.01
- added link tool0
- added link world
Joints:
- added joint base_link-base_fixed_joint: type fixed, parent base_link, child base, origin xyz=0 0 0 rpy=0 0 -3.1415926536
- added joint ee_fixed_joint: type fixed, parent wrist_3_link, child ee_link, origin xyz=0.0 0.04436 0.0 rpy=0.0 0.0 1.57079632679
- added joint world_joint: type fixed, parent world, child base_link, origin xyz=0.0 0.0 0.0 rpy=3.1415926536 3.1415926536 0.0
- added joint wrist_3_link-tool0_fixed_joint: type fixed, parent wrist_3_link, child tool0, origin xyz=0 0.04436 0 rpy=-1.57079632679 0 0
